Commit message: fix xacro warning
  deprecated: xacro tags should be prepended with 'xacro' xml namespace.
    Use the following script to fix incorrect usage:
              find . -iname "*.xacro" | xargs sed -i 's#<\([/]\?\)\(if\|unless\|include\|arg\|property\|macro\|insert_block\)#<\1xacro:\2#g'

File: pal_gripper_description/gazebo/gazebo.urdf.xacro (robot description, xacro)
@@ -17,4 +17,4 @@
   </gazebo>
   <!-- define global properties -->
-  <property name="M_PI" value="3.1415926535897931" />
+  <xacro:property name="M_PI" value="3.1415926535897931" />
 </robot>

File: pal_gripper_description/urdf/deg_to_rad.urdf.xacro (robot description, xacro)
@@ -1,3 +1,3 @@
 <robot xmlns:xacro="http://ros.org/wiki/xacro">
-	<property name="deg_to_rad" value="0.01745329251994329577" />
+	<xacro:property name="deg_to_rad" value="0.01745329251994329577" />
 </robot>

File: pal_gripper_description/urdf/gripper.urdf.xacro (robot description, xacro)
@@ -17,5 +17,5 @@
   </link>
   <joint name="${name}_tool_joint" type="fixed">
-    <insert_block name="origin"/>
+    <xacro:insert_block name="origin"/>
     <parent link="${parent}" />
     <child link="${name}_tool_link" />
@@ -48,5 +48,5 @@
   </gazebo>
   <joint name="${name}_joint" type="fixed">
-    <insert_block name="origin"/>
+    <xacro:insert_block name="origin"/>
     <parent link="${parent}" />
     <child link="${name}_link" />

Commit message: rm usuless xacro property

File: pal_gripper_description/gazebo/gazebo.urdf.xacro (robot description, xacro)
@@ -16,5 +16,3 @@
     </plugin>
   </gazebo>
-  <!-- define global properties -->
-  <xacro:property name="M_PI" value="3.1415926535897931" />
 </robot>
