Commit message: remove grasping hack macro and tune friction

File: pal_gripper_description/urdf/gripper.gazebo.xacro (robot description, xacro)
@@ -8,33 +8,13 @@
 -->
 <robot xmlns:xacro="http://ros.org/wiki/xacro">
-    <xacro:macro name="gripper_grasping_hack" params="name">
-      <gazebo>
-        <gripper name="${name}_grasp_hack">
-          <grasp_check>
-            <attach_steps>1</attach_steps>
-            <detach_steps>2</detach_steps>
-            <min_contact_count>2</min_contact_count>
-          </grasp_check>
-          <gripper_link>${name}_left_finger_link</gripper_link>
-          <gripper_link>${name}_right_finger_link</gripper_link>
-          <palm_link>${name}_link</palm_link>
-        </gripper>
-      </gazebo>
-    </xacro:macro>
-    <xacro:macro name="finger_gazebo" params="name">
-<!--
-    <gazebo reference="${finger_name}_link">
-      <mu1>0.9</mu1>
-      <mu2>0.9</mu2>
-    </gazebo>
--->
+  <xacro:macro name="finger_gazebo" params="name">
     <gazebo reference="${name}_link">
       <kp>1000000.0</kp>
-      <kd>100.0</kd>
+      <kd>1.0</kd>
       <mu1>1.0</mu1>
       <mu2>1.0</mu2>
-      <fdir1>0 0 1</fdir1>
+      <fdir1>0 0 0</fdir1>
       <maxVel>1.0</maxVel>
-      <minDepth>0.00</minDepth>
+      <minDepth>0.1</minDepth>
       <material>Gazebo/Black</material>
     </gazebo>

Commit message: Improve grasping in simulation and on real robot + change is_grasped topic name

File: pal_gripper_description/urdf/gripper.gazebo.xacro (robot description, xacro)
@@ -10,11 +10,28 @@
   <xacro:macro name="finger_gazebo" params="name">
     <gazebo reference="${name}_link">
-      <kp>1000000.0</kp>
-      <kd>1.0</kd>
-      <mu1>1.0</mu1>
-      <mu2>1.0</mu2>
-      <fdir1>0 0 0</fdir1>
-      <maxVel>1.0</maxVel>
-      <minDepth>0.1</minDepth>
+      <collision name="${name}_link">
+        <surface>
+          <friction>
+            <torsional>
+              <coefficient>1000.0</coefficient>
+              <use_patch_radius>true</use_patch_radius>
+              <patch_radius>0.1</patch_radius>
+            </torsional>
+          </friction>
+          <contact>
+            <poissons_ratio>1.0</poissons_ratio>
+            <elastic_modulus>Inf</elastic_modulus>
+          </contact>
+        </surface>
+      </collision>
+      <mu1>Inf</mu1>
+      <mu2>Inf</mu2>
+      <maxVel>0.0</maxVel>
+      <kp>Inf</kp>
+      <kd>100.0</kd>
+      <fdir1>1 0 0</fdir1>
+      <maxVel>0.0</maxVel>
+      <minDepth>0.002</minDepth>
+      <maxContacts>100</maxContacts>
       <material>Gazebo/Black</material>
     </gazebo>
