Commit message: ros2 update transmissions for pal-gripper

File: pal_gripper_description/urdf/gripper.ros2_control.xacro (robot description, xacro)
@@ -20,16 +20,6 @@
       <state_interface name="effort" />
     </joint>
-    <!-- @TODO transmissions for ros2 system -->
-    <!--
-    <transmission name="${name}_trans">
-      <type>transmission_interface/SimpleTransmission</type>
-      <actuator name="${name}_motor" >
-        <mechanicalReduction>${reduction}</mechanicalReduction>
-      </actuator>
-      <joint name="${name}_joint">
-        <hardwareInterface>hardware_interface/PositionJointInterface</hardwareInterface>
-      </joint>
-    </transmission>
-    -->
+    <xacro:include filename="$(find pal_gripper_description)/urdf/gripper.transmission.xacro" />
+    <xacro:gripper_simple_transmission name="${name}" reduction="${reduction}" />
   </xacro:macro>
 </robot>

File: pal_gripper_description/urdf/gripper.transmission.xacro (robot description, xacro)
@@ -13,12 +13,10 @@
  -->
 <robot xmlns:xacro="http://ros.org/wiki/xacro">
-  <xacro:macro name="gripper_simple_transmission" params="name reduction" >
+  <xacro:macro name="gripper_simple_transmission" params="name reduction">
     <transmission name="${name}_trans">
-      <type>transmission_interface/SimpleTransmission</type>
-      <actuator name="${name}_motor" >
-        <mechanicalReduction>${reduction}</mechanicalReduction>
-      </actuator>
-      <joint name="${name}_joint">
-        <hardwareInterface>hardware_interface/PositionJointInterface</hardwareInterface>
+      <plugin>transmission_interface/SimpleTransmission</plugin>
+      <actuator name="${name}_motor" role="actuator1"/>
+      <joint name="${name}_joint" role="joint1">
+        <mechanical_reduction>${reduction}</mechanical_reduction>
       </joint>
     </transmission>

File: pal_gripper_description/urdf/gripper.urdf.xacro (robot description, xacro)
@@ -3,5 +3,4 @@
   <!--File includes-->
   <xacro:include filename="$(find pal_gripper_description)/urdf/deg_to_rad.urdf.xacro" />
-  <xacro:include filename="$(find pal_gripper_description)/urdf/gripper.transmission.xacro" />
   <xacro:include filename="$(find pal_gripper_description)/urdf/gripper.gazebo.xacro" />
   <xacro:property name="gripper_eps" value="0.001" />
@@ -144,6 +143,4 @@
     </inertial>
   </link>
-  <xacro:gripper_simple_transmission name="${name}_left_finger" reduction="1.0"/>
-  <xacro:gripper_simple_transmission name="${name}_right_finger" reduction="1.0"/>
   <xacro:finger_gazebo name="${name}_left_finger"/>
   <xacro:finger_gazebo name="${name}_right_finger"/>
