Commit message: Added safety controller values

File: pal_gripper_description/urdf/gripper.urdf.xacro (robot description, xacro)
@@ -5,4 +5,5 @@
   <xacro:include filename="$(find pal_gripper_description)/urdf/gripper.transmission.xacro" />
   <xacro:include filename="$(find pal_gripper_description)/urdf/gripper.gazebo.xacro" />
+  <xacro:property name="gripper_eps" value="0.001" />
   <xacro:macro name="pal_gripper" params="name parent *origin">
   <link name="${name}_link">
@@ -70,4 +71,8 @@
     <calibration rising="0.0" />
     <dynamics damping="2500" />
+    <safety_controller k_position="20"
+                       k_velocity="20"
+                       soft_lower_limit="${0.0 * deg_to_rad + gripper_eps}"
+                       soft_upper_limit="${0.048 * deg_to_rad - gripper_eps}" />
   </joint>
   <link name="${name}_left_finger_link">
@@ -104,4 +109,8 @@
     <calibration rising="0.0" />
     <dynamics damping="2500" />
+    <safety_controller k_position="20"
+                       k_velocity="20"
+                       soft_lower_limit="${0.0 * deg_to_rad + gripper_eps}"
+                       soft_upper_limit="${0.048 * deg_to_rad - gripper_eps}" />
   </joint>
   <!-- Grasping frame -->

Commit message: Change gripper limit to 0.045

File: pal_gripper_description/urdf/gripper.urdf.xacro (robot description, xacro)
@@ -68,5 +68,5 @@
     <child link="${name}_right_finger_link" />
     <axis xyz="1 0 0" />
-    <limit effort="28.0" lower="0.0" upper="0.048" velocity="0.1" />
+    <limit effort="28.0" lower="0.0" upper="0.045" velocity="0.1" />
     <calibration rising="0.0" />
     <dynamics damping="2500" />
@@ -74,5 +74,5 @@
                        k_velocity="20"
                        soft_lower_limit="${0.0 + gripper_eps}"
-                       soft_upper_limit="${0.048 - gripper_eps}" />
+                       soft_upper_limit="${0.045 - gripper_eps}" />
   </joint>
   <link name="${name}_left_finger_link">
@@ -106,5 +106,5 @@
     <child link="${name}_left_finger_link" />
     <axis xyz="-1 0 0" />
-    <limit effort="28.0" lower="0" upper="0.048" velocity="0.1" />
+    <limit effort="28.0" lower="0" upper="0.045" velocity="0.1" />
     <calibration rising="0.0" />
     <dynamics damping="2500" />
@@ -112,5 +112,5 @@
                        k_velocity="20"
                        soft_lower_limit="${0.0 + gripper_eps}"
-                       soft_upper_limit="${0.048 - gripper_eps}" />
+                       soft_upper_limit="${0.045 - gripper_eps}" />
   </joint>
   <!-- Grasping frame -->

Commit message: update meshes and inertia matrices

File: pal_gripper_description/urdf/gripper.urdf.xacro (robot description, xacro)
@@ -9,9 +9,9 @@
   <link name="${name}_link">
     <inertial>
-      <origin rpy="0.0 0.0 0.0" xyz="-0.00028 0.00028 -0.03963" />
-      <mass value="0.71" />
-      <inertia ixx="0.00205962" ixy="0" ixz="0"
-               iyy="0.00250896" iyz="0"
-               izz="0.00086580" />
+      <origin rpy="0.0 0.0 0.0" xyz="-0.000294 0.000291 -0.033086" />
+      <mass value="0.602660" />
+      <inertia ixx="0.000693" ixy="0.000045" ixz="-0.000000"
+               iyy="0.001024" iyz="0.000000"
+               izz="0.000672" />
     </inertial>
     <visual>
@@ -40,12 +40,12 @@
   <link name="${name}_right_finger_link">
     <inertial>
-      <origin rpy="0 0 0" xyz="-0.00402 0.04101 0.01061" />
-      <mass value="0.06" />
-      <inertia ixx="0.00018039" ixy="0" ixz="0"
-               iyy="0.00002373" iyz="0"
-               izz="0.00018646" />
+      <origin rpy="0 0 0" xyz="-0.004470 0.010766 -0.121013" />
+      <mass value="0.109980" />
+      <inertia ixx="0.000232" ixy="-0.000005" ixz="-0.000032"
+               iyy="0.000224" iyz="0.000036"
+               izz="0.000029" />
     </inertial>
     <visual>
-      <origin rpy="0 0 0" xyz="-0.049 0 0" />
+      <origin rpy="0 0 3.1415" xyz="0 0 0" />
       <geometry>
         <mesh filename="package://pal_gripper_description/meshes/gripper_finger_link.stl" scale="-1 -1 1"/>
@@ -54,5 +54,5 @@
     </visual>
     <collision>
-      <origin rpy="0 0 0" xyz="-0.049 0 0" />
+      <origin rpy="0 0 3.1415" xyz="0 0 0" />
       <geometry>
         <mesh filename="package://pal_gripper_description/meshes/gripper_finger_link_collision.stl" scale="-1 -1 1"/>
@@ -68,7 +68,7 @@
     <child link="${name}_right_finger_link" />
     <axis xyz="1 0 0" />
-    <limit effort="28.0" lower="0.0" upper="0.045" velocity="0.1" />
+    <limit effort="16" lower="0.0" upper="0.045" velocity="0.05" />
     <calibration rising="0.0" />
-    <dynamics damping="2500" />
+    <dynamics damping="80" />
     <safety_controller k_position="20"
                        k_velocity="20"
@@ -78,12 +78,12 @@
   <link name="${name}_left_finger_link">
     <inertial>
-      <origin rpy="0 0 0" xyz="-0.00402 0.04101 0.01061" />
-      <mass value="0.06" />
-      <inertia ixx="0.00018039" ixy="0" ixz="0"
-               iyy="0.00002373" iyz="0"
-               izz="0.00018646" />
+      <origin rpy="0 0 0" xyz="-0.004470 0.010766 -0.121013" />
+      <mass value="0.109980" />
+      <inertia ixx="0.000232" ixy="-0.000005" ixz="-0.000032"
+               iyy="0.000224" iyz="0.000036"
+               izz="0.000029" />
     </inertial>
     <visual>
-      <origin rpy="0 0 0" xyz="0.049 0 0"/>
+      <origin rpy="0 0 3.1415" xyz="0 0 0"/>
       <geometry>
         <mesh filename="package://pal_gripper_description/meshes/gripper_finger_link.stl"/>
@@ -92,5 +92,5 @@
     </visual>
     <collision>
-      <origin rpy="0 0 0" xyz="0.049 0 0" />
+      <origin rpy="0 0 3.1415" xyz="0 0 0" />
       <geometry>
         <mesh filename="package://pal_gripper_description/meshes/gripper_finger_link_collision.stl"/>
@@ -106,7 +106,7 @@
     <child link="${name}_left_finger_link" />
     <axis xyz="-1 0 0" />
-    <limit effort="28.0" lower="0" upper="0.045" velocity="0.1" />
+    <limit effort="16" lower="0" upper="0.045" velocity="0.05" />
     <calibration rising="0.0" />
-    <dynamics damping="2500" />
+    <dynamics damping="80" />
     <safety_controller k_position="20"
                        k_velocity="20"
@@ -133,5 +133,4 @@
   <xacro:finger_gazebo name="${name}_left_finger"/>
   <xacro:finger_gazebo name="${name}_right_finger"/>
-  <xacro:gripper_grasping_hack name="${name}"/>
  </xacro:macro>
 </robot>

Commit message: use box for fingers' collision model

File: pal_gripper_description/urdf/gripper.urdf.xacro (robot description, xacro)
@@ -54,7 +54,7 @@
     </visual>
     <collision>
-      <origin rpy="0 0 3.1415" xyz="0 0 0" />
+      <origin rpy="0 0 3.1415" xyz="0.005 0 -0.165" />
       <geometry>
-        <mesh filename="package://pal_gripper_description/meshes/gripper_finger_link_collision.stl" scale="-1 -1 1"/>
+        <box size="0.01 0.05 0.11"/>
       </geometry>
     </collision>
@@ -92,7 +92,7 @@
     </visual>
     <collision>
-      <origin rpy="0 0 3.1415" xyz="0 0 0" />
+      <origin rpy="0 0 3.1415" xyz="-0.005 0 -0.165" />
       <geometry>
-        <mesh filename="package://pal_gripper_description/meshes/gripper_finger_link_collision.stl"/>
+        <box size="0.01 0.05 0.11"/>
       </geometry>
     </collision>

Commit message: Fixed problem with gripper_grasping_frame in wrong position

File: pal_gripper_description/urdf/gripper.urdf.xacro (robot description, xacro)
@@ -118,5 +118,5 @@
     <parent link="${name}_link" />
     <child link="${name}_grasping_frame" />
-    <origin xyz="0.12 0 0" rpy="0 0 0" />
+    <origin xyz="0 0 -0.12" rpy="-1.5708 1.5708 0" />
   </joint>
   <link name="${name}_grasping_frame">

Commit message: Add tool link

File: pal_gripper_description/urdf/gripper.urdf.xacro (robot description, xacro)
@@ -7,4 +7,19 @@
   <xacro:property name="gripper_eps" value="0.001" />
   <xacro:macro name="pal_gripper" params="name parent *origin">
+  <link name="${name}_tool_link">
+    <inertial>
+      <origin xyz="0 0 0" rpy="0 0 0" />
+      <mass value="0.0001" />
+      <inertia ixx="0.00001" ixy="0.0" ixz="0.0"
+               iyy="0.00001" iyz="0.0"
+               izz="0.00001" />
+    </inertial>
+  </link>
+  <joint name="${name}_tool_joint" type="fixed">
+    <insert_block name="origin"/>
+    <parent link="${parent}" />
+    <child link="${name}_tool_link" />
+    <axis xyz="0 0 0" />
+  </joint>
   <link name="${name}_link">
     <inertial>

Commit message: remove link color discrepancy

File: pal_gripper_description/urdf/gripper.urdf.xacro (robot description, xacro)
@@ -66,5 +66,5 @@
         <mesh filename="package://pal_gripper_description/meshes/gripper_finger_link.stl" scale="-1 -1 1"/>
       </geometry>
-      <material name="White"/>
+      <material name="Black"/>
     </visual>
     <collision>
@@ -76,5 +76,5 @@
   </link>
   <gazebo reference="${name}_right_finger_link">
-    <material>Gazebo/White</material>
+    <material>Gazebo/Black</material>
   </gazebo>
   <joint name="${name}_right_finger_joint" type="prismatic">
@@ -104,5 +104,5 @@
         <mesh filename="package://pal_gripper_description/meshes/gripper_finger_link.stl"/>
       </geometry>
-      <material name="White"/>
+      <material name="Black"/>
     </visual>
     <collision>
@@ -114,5 +114,5 @@
   </link>
   <gazebo reference="${name}_left_finger_link">
-    <material>Gazebo/White</material>
+    <material>Gazebo/Black</material>
   </gazebo>
   <joint name="${name}_left_finger_joint" type="prismatic">

Commit message: add friction to gripper fingers

File: pal_gripper_description/urdf/gripper.urdf.xacro (robot description, xacro)
@@ -85,5 +85,5 @@
     <limit effort="16" lower="0.0" upper="0.045" velocity="0.05" />
     <calibration rising="0.0" />
-    <dynamics damping="80" />
+    <dynamics damping="80" friction="2.0"/>
     <safety_controller k_position="20"
                        k_velocity="20"
@@ -123,5 +123,5 @@
     <limit effort="16" lower="0" upper="0.045" velocity="0.05" />
     <calibration rising="0.0" />
-    <dynamics damping="80" />
+    <dynamics damping="80" friction="2.0"/>
     <safety_controller k_position="20"
                        k_velocity="20"

Commit message: Add grasp_hack + tuning

File: pal_gripper_description/urdf/gripper.urdf.xacro (robot description, xacro)
@@ -7,4 +7,18 @@
   <xacro:property name="gripper_eps" value="0.001" />
   <xacro:macro name="pal_gripper" params="name parent *origin">
+  <xacro:macro name="grasp_hack_parallel" params="hack_name name_prefix_left name_prefix_right parent_joint">
+    <gazebo>
+      <gripper name="${hack_name}">
+        <grasp_check>
+          <attach_steps>1</attach_steps>
+          <detach_steps>1</detach_steps>    <!-- should be higher than 1 otherwise the object will be attached to the gripper too much time -->
+          <min_contact_count>3</min_contact_count>
+        </grasp_check>
+        <gripper_link>${name_prefix_left}</gripper_link>
+        <gripper_link>${name_prefix_right}</gripper_link>
+        <palm_link>${parent_joint}</palm_link>
+      </gripper>
+    </gazebo>
+  </xacro:macro>
   <link name="${name}_tool_link">
     <inertial>
@@ -83,7 +97,7 @@
     <child link="${name}_right_finger_link" />
     <axis xyz="1 0 0" />
-    <limit effort="16" lower="0.0" upper="0.045" velocity="0.05" />
+    <limit effort="64" lower="0.0" upper="0.045" velocity="0.05" />
     <calibration rising="0.0" />
-    <dynamics damping="80" />
+    <dynamics damping="1" />
     <safety_controller k_position="20"
                        k_velocity="20"
@@ -121,7 +135,7 @@
     <child link="${name}_left_finger_link" />
     <axis xyz="-1 0 0" />
-    <limit effort="16" lower="0" upper="0.045" velocity="0.05" />
+    <limit effort="64" lower="0" upper="0.045" velocity="0.05" />
     <calibration rising="0.0" />
-    <dynamics damping="80" />
+    <dynamics damping="1" />
     <safety_controller k_position="20"
                        k_velocity="20"
@@ -146,4 +160,5 @@
   <xacro:gripper_simple_transmission name="${name}_left_finger" reduction="1.0"/>
   <xacro:gripper_simple_transmission name="${name}_right_finger" reduction="1.0"/>
+  <xacro:grasp_hack_parallel hack_name="${name}_grasp_hack" name_prefix_left="${name}_left_finger_link" name_prefix_right="${name}_right_finger_link" parent_joint="${parent}"/>
   <xacro:finger_gazebo name="${name}_left_finger"/>
   <xacro:finger_gazebo name="${name}_right_finger"/>

Commit message: Apply Sai suggestion for naming and syntax

File: pal_gripper_description/urdf/gripper.urdf.xacro (robot description, xacro)
@@ -7,7 +7,7 @@
   <xacro:property name="gripper_eps" value="0.001" />
   <xacro:macro name="pal_gripper" params="name parent *origin">
-  <xacro:macro name="grasp_hack_parallel" params="hack_name name_prefix_left name_prefix_right parent_joint">
+  <xacro:macro name="gazebo_gripper_grasp" params="name name_prefix_left name_prefix_right parent_joint">
     <gazebo>
-      <gripper name="${hack_name}">
+      <gripper name="${name}">
         <grasp_check>
           <attach_steps>1</attach_steps>
@@ -160,5 +160,5 @@
   <xacro:gripper_simple_transmission name="${name}_left_finger" reduction="1.0"/>
   <xacro:gripper_simple_transmission name="${name}_right_finger" reduction="1.0"/>
-  <xacro:grasp_hack_parallel hack_name="${name}_grasp_hack" name_prefix_left="${name}_left_finger_link" name_prefix_right="${name}_right_finger_link" parent_joint="${parent}"/>
+  <xacro:gazebo_gripper_grasp name="${name}_grasp" name_prefix_left="${name}_left_finger_link" name_prefix_right="${name}_right_finger_link" parent_joint="${parent}"/>
   <xacro:finger_gazebo name="${name}_left_finger"/>
   <xacro:finger_gazebo name="${name}_right_finger"/>

Commit message: Added grasping frame Z and Y

File: pal_gripper_description/urdf/gripper.urdf.xacro (robot description, xacro)
@@ -158,4 +158,34 @@
     </inertial>
   </link>
+  <!-- Grasping frame Y -->
+  <joint name="${name}_grasping_frame_Y_joint" type="fixed">
+    <parent link="${name}_link" />
+    <child link="${name}_grasping_frame_Y" />
+    <origin xyz="0 0 -0.12" rpy="-1.5708 0 1.5708" />
+  </joint>
+  <link name="${name}_grasping_frame_Y">
+    <inertial>
+      <origin xyz="0 0 0" rpy="0 0 0" />
+      <mass value="0.0001" />
+      <inertia ixx="0.00001" ixy="0.0" ixz="0.0"
+               iyy="0.00001" iyz="0.0"
+               izz="0.00001" />
+    </inertial>
+  </link>
+  <!-- Grasping frame Z -->
+  <joint name="${name}_grasping_frame_Z_joint" type="fixed">
+    <parent link="${name}_link" />
+    <child link="${name}_grasping_frame_Z" />
+    <origin xyz="0 0 -0.12" rpy="3.1416 0 1.5708" />
+  </joint>
+  <link name="${name}_grasping_frame_Z">
+    <inertial>
+      <origin xyz="0 0 0" rpy="0 0 0" />
+      <mass value="0.0001" />
+      <inertia ixx="0.00001" ixy="0.0" ixz="0.0"
+               iyy="0.00001" iyz="0.0"
+               izz="0.00001" />
+    </inertial>
+  </link>
   <xacro:gripper_simple_transmission name="${name}_left_finger" reduction="1.0"/>
   <xacro:gripper_simple_transmission name="${name}_right_finger" reduction="1.0"/>

Commit message: Added gripper base link

File: pal_gripper_description/urdf/gripper.urdf.xacro (robot description, xacro)
@@ -67,4 +67,10 @@
     <axis xyz="0 0 0" />
   </joint>
+  <link name="${name}_base_link"/>
+  <joint name="${name}_base_joint" type="fixed">
+    <origin rpy="0 3.1416 1.5707" xyz="0. 0 0" />
+    <parent link="${name}_link" />
+    <child link="${name}_base_link" />
+  </joint>
   <link name="${name}_right_finger_link">
     <inertial>

Commit message: Replaced links by grasping frame macro

File: pal_gripper_description/urdf/gripper.urdf.xacro (robot description, xacro)
@@ -5,4 +5,5 @@
   <xacro:include filename="$(find pal_gripper_description)/urdf/gripper.transmission.xacro" />
   <xacro:include filename="$(find pal_gripper_description)/urdf/gripper.gazebo.xacro" />
+  <xacro:include filename="$(find tiago_description)/urdf/end_effector/grasping_frames.xacro" />
   <xacro:property name="gripper_eps" value="0.001" />
   <xacro:macro name="pal_gripper" params="name parent *origin">
@@ -149,49 +150,5 @@
                        soft_upper_limit="${0.045 - gripper_eps}" />
   </joint>
-  <!-- Grasping frame -->
-  <joint name="${name}_grasping_frame_joint" type="fixed">
-    <parent link="${name}_link" />
-    <child link="${name}_grasping_frame" />
-    <origin xyz="0 0 -0.12" rpy="-1.5708 1.5708 0" />
-  </joint>
-  <link name="${name}_grasping_frame">
-    <inertial>
-      <origin xyz="0 0 0" rpy="0 0 0" />
-      <mass value="0.0001" />
-      <inertia ixx="0.00001" ixy="0.0" ixz="0.0"
-               iyy="0.00001" iyz="0.0"
-               izz="0.00001" />
-    </inertial>
-  </link>
-  <!-- Grasping frame Y -->
-  <joint name="${name}_grasping_frame_Y_joint" type="fixed">
-    <parent link="${name}_link" />
-    <child link="${name}_grasping_frame_Y" />
-    <origin xyz="0 0 -0.12" rpy="-1.5708 0 1.5708" />
-  </joint>
-  <link name="${name}_grasping_frame_Y">
-    <inertial>
-      <origin xyz="0 0 0" rpy="0 0 0" />
-      <mass value="0.0001" />
-      <inertia ixx="0.00001" ixy="0.0" ixz="0.0"
-               iyy="0.00001" iyz="0.0"
-               izz="0.00001" />
-    </inertial>
-  </link>
-  <!-- Grasping frame Z -->
-  <joint name="${name}_grasping_frame_Z_joint" type="fixed">
-    <parent link="${name}_link" />
-    <child link="${name}_grasping_frame_Z" />
-    <origin xyz="0 0 -0.12" rpy="3.1416 0 1.5708" />
-  </joint>
-  <link name="${name}_grasping_frame_Z">
-    <inertial>
-      <origin xyz="0 0 0" rpy="0 0 0" />
-      <mass value="0.0001" />
-      <inertia ixx="0.00001" ixy="0.0" ixz="0.0"
-               iyy="0.00001" iyz="0.0"
-               izz="0.00001" />
-    </inertial>
-  </link>
+  <xacro:pal_robotiq_grasping_frames prefix="${name}_" xyz="0 0 0.12"/>
   <xacro:gripper_simple_transmission name="${name}_left_finger" reduction="1.0"/>
   <xacro:gripper_simple_transmission name="${name}_right_finger" reduction="1.0"/>

Commit message: Fix finger position

File: pal_gripper_description/urdf/gripper.urdf.xacro (robot description, xacro)
@@ -70,5 +70,5 @@
   </gazebo>
   <joint name="${name}_right_finger_joint" type="prismatic">
-    <origin rpy="0 0 0" xyz="0 0 0.01" />
+    <origin rpy="0 0 0" xyz="0 0 -0.01" />
     <parent link="${name}_link" />
     <child link="${name}_right_finger_link" />
@@ -108,5 +108,5 @@
   </gazebo>
   <joint name="${name}_left_finger_joint" type="prismatic">
-    <origin rpy="0 0 0" xyz="0 0 0.01" />
+    <origin rpy="0 0 0" xyz="0 0 -0.01" />
     <parent link="${name}_link" />
     <child link="${name}_left_finger_link" />

Commit message: Change the way of finding packages for meshes

File: pal_gripper_description/urdf/gripper.urdf.xacro (robot description, xacro)
@@ -24,5 +24,5 @@
       <origin rpy="0 0 0" xyz="0 0 0" />
       <geometry>
-        <mesh filename="package://pal_gripper_description/meshes/gripper_link.stl"/>
+        <mesh filename="file://$(find pal_gripper_description)/meshes/gripper_link.stl"/>
       </geometry>
       <material name="White"/>
@@ -31,5 +31,5 @@
       <origin rpy="0 0 0" xyz="0 0 0" />
       <geometry>
-        <mesh filename="package://pal_gripper_description/meshes/gripper_link_collision.stl"/>
+        <mesh filename="file://$(find pal_gripper_description)/meshes/gripper_link_collision.stl"/>
       </geometry>
     </collision>
@@ -55,5 +55,5 @@
       <origin rpy="0 0 3.1415" xyz="0 0 0" />
       <geometry>
-        <mesh filename="package://pal_gripper_description/meshes/gripper_finger_link.stl" scale="-1 -1 1"/>
+        <mesh filename="file://$(find pal_gripper_description)/meshes/gripper_finger_link.stl" scale="-1 -1 1"/>
       </geometry>
       <material name="Black"/>
@@ -93,5 +93,5 @@
       <origin rpy="0 0 3.1415" xyz="0 0 0"/>
       <geometry>
-        <mesh filename="package://pal_gripper_description/meshes/gripper_finger_link.stl"/>
+        <mesh filename="file://$(find pal_gripper_description)/meshes/gripper_finger_link.stl"/>
       </geometry>
       <material name="Black"/>

Commit message: Add support for new gazebo

File: pal_gripper_description/urdf/gripper.urdf.xacro (robot description, xacro)
@@ -69,4 +69,12 @@
     <material>Gazebo/Black</material>
   </gazebo>
+  <!-- TODO: set lower limit back to 0 when moving to Gazebo Harmonic or ROS 2 Jazzy -->
+  <!-- See https://github.com/gazebosim/gz-sim/issues/1684 for more information -->
+  <xacro:if value="${gazebo_version == 'classic'}">
+    <xacro:property name="gripper_lower_limit" value="0.0"/>
+  </xacro:if>
+  <xacro:if value="${gazebo_version == 'gazebo'}">
+    <xacro:property name="gripper_lower_limit" value="-1e-3"/>
+  </xacro:if>
   <joint name="${name}_right_finger_joint" type="prismatic">
     <origin rpy="0 0 0" xyz="0 0 -0.01" />
@@ -74,5 +82,5 @@
     <child link="${name}_right_finger_link" />
     <axis xyz="1 0 0" />
-    <limit effort="16" lower="0.0" upper="0.045" velocity="0.05" />
+    <limit effort="16" lower="${gripper_lower_limit}" upper="0.045" velocity="0.05" />
     <calibration rising="0.0" />
     <dynamics damping="80" friction="2.0"/>
@@ -112,5 +120,5 @@
     <child link="${name}_left_finger_link" />
     <axis xyz="-1 0 0" />
-    <limit effort="16" lower="0" upper="0.045" velocity="0.05" />
+    <limit effort="16" lower="${gripper_lower_limit}" upper="0.045" velocity="0.05" />
     <calibration rising="0.0" />
     <dynamics damping="80" friction="2.0"/>

Commit message: Use package instead of find for meshes lookup
This change avoids errors when visualizing the robot in rviz2 from a
remote host instead of directly inside the robot

File: pal_gripper_description/urdf/gripper.urdf.xacro (robot description, xacro)
@@ -24,5 +24,5 @@
       <origin rpy="0 0 0" xyz="0 0 0" />
       <geometry>
-        <mesh filename="file://$(find pal_gripper_description)/meshes/gripper_link.stl"/>
+        <mesh filename="package://pal_gripper_description/meshes/gripper_link.stl"/>
       </geometry>
       <material name="White"/>
@@ -31,5 +31,5 @@
       <origin rpy="0 0 0" xyz="0 0 0" />
       <geometry>
-        <mesh filename="file://$(find pal_gripper_description)/meshes/gripper_link_collision.stl"/>
+        <mesh filename="package://pal_gripper_description/meshes/gripper_link_collision.stl"/>
       </geometry>
     </collision>
@@ -55,5 +55,5 @@
       <origin rpy="0 0 3.1415" xyz="0 0 0" />
       <geometry>
-        <mesh filename="file://$(find pal_gripper_description)/meshes/gripper_finger_link.stl" scale="-1 -1 1"/>
+        <mesh filename="package://pal_gripper_description/meshes/gripper_finger_link.stl" scale="-1 -1 1"/>
       </geometry>
       <material name="Black"/>
@@ -93,5 +93,5 @@
       <origin rpy="0 0 3.1415" xyz="0 0 0"/>
       <geometry>
-        <mesh filename="file://$(find pal_gripper_description)/meshes/gripper_finger_link.stl"/>
+        <mesh filename="package://pal_gripper_description/meshes/gripper_finger_link.stl"/>
       </geometry>
       <material name="Black"/>
