Commit message: Added a gazebo model launch with controller to test that the gripper opens and closes

File: pal_gripper_description/robots/gripper_test.urdf.xacro (robot description, xacro)
@@ -12,8 +12,10 @@
   <xacro:include filename="$(find pal_gripper_description)/urdf/deg_to_rad.urdf.xacro" />
   <xacro:include filename="$(find pal_gripper_description)/urdf/gripper.urdf.xacro" />
+  <!-- Generic simulator_gazebo plugins -->
+  <xacro:include filename="$(find pal_gripper_description)/gazebo/gazebo.urdf.xacro" />
   <!--Spawn gripper-->
   <link name="base_link"/>
   <xacro:pal_gripper parent="base_link" name="gripper">
-    <origin xyz="0 0 0" rpy="0 ${90 * deg_to_rad} ${90 * deg_to_rad}" />
+    <origin xyz="0 0 0" rpy="0 ${180 * deg_to_rad} ${0 * deg_to_rad}" />
   </xacro:pal_gripper>
 </robot>

File: pal_gripper_description/urdf/gripper.urdf.xacro (robot description, xacro)
@@ -5,4 +5,5 @@
   <xacro:include filename="$(find pal_gripper_description)/urdf/gripper.transmission.xacro" />
   <xacro:include filename="$(find pal_gripper_description)/urdf/gripper.gazebo.xacro" />
+  <xacro:include filename="$(find pal_gripper_description)/urdf/materials.urdf.xacro" />
   <xacro:macro name="pal_gripper" params="name parent *origin">
   <link name="${name}_link">
@@ -19,5 +20,5 @@
         <mesh filename="package://pal_gripper_description/meshes/gripper_link.stl"/>
       </geometry>
-      <!-- <material name="White"/> -->
+      <material name="White"/>
     </visual>
     <collision>
@@ -46,12 +47,12 @@
     </inertial>
     <visual>
-      <origin rpy="0 0 0" xyz="-0.048 0 0" />
+      <origin rpy="0 0 0" xyz="-0.049 0 0" />
       <geometry>
         <mesh filename="package://pal_gripper_description/meshes/gripper_finger_link.stl" scale="-1 -1 1"/>
       </geometry>
-      <!-- <material name="Black"/> -->
+      <material name="White"/>
     </visual>
     <collision>
-      <origin rpy="0 0 0" xyz="-0.048 0 0" />
+      <origin rpy="0 0 0" xyz="-0.049 0 0" />
       <geometry>
         <mesh filename="package://pal_gripper_description/meshes/gripper_finger_link_collision.stl" scale="-1 -1 1"/>
@@ -59,4 +60,7 @@
     </collision>
   </link>
+  <gazebo reference="${name}_right_finger_link">
+    <material>Gazebo/White</material>
+  </gazebo>
   <joint name="${name}_right_finger_joint" type="prismatic">
     <origin rpy="0 0 0" xyz="0. 0 0" />
@@ -77,12 +81,12 @@
     </inertial>
     <visual>
-      <origin rpy="0 0 0" xyz="0.048 0 0"/>
+      <origin rpy="0 0 0" xyz="0.049 0 0"/>
       <geometry>
         <mesh filename="package://pal_gripper_description/meshes/gripper_finger_link.stl"/>
       </geometry>
-      <!-- <material name="Black"/> -->
+      <material name="White"/>
     </visual>
     <collision>
-      <origin rpy="0 0 0" xyz="0.048 0 0" />
+      <origin rpy="0 0 0" xyz="0.049 0 0" />
       <geometry>
         <mesh filename="package://pal_gripper_description/meshes/gripper_finger_link_collision.stl"/>
@@ -90,4 +94,7 @@
     </collision>
   </link>
+  <gazebo reference="${name}_left_finger_link">
+    <material>Gazebo/White</material>
+  </gazebo>
   <joint name="${name}_left_finger_joint" type="prismatic">
     <origin rpy="0 0 0" xyz="0. 0 0" />

Commit message: add calibration tool

File: pal_gripper_description/robots/gripper_test.urdf.xacro (robot description, xacro)
@@ -14,4 +14,6 @@
 <robot xmlns:xacro="http://ros.org/wiki/xacro"
        name="pal_gripper">
+  <!-- Properties-->
+  <xacro:property name="calibration_tool" value="$(arg calibration_tool)" />
   <!--External resources-->
   <xacro:include filename="$(find pal_urdf_utils)/urdf/deg_to_rad.urdf.xacro" />
@@ -32,5 +34,5 @@
   <!--Spawn gripper-->
   <link name="base_link"/>
-  <xacro:pal_gripper parent="base_link" name="gripper">
+  <xacro:pal_gripper parent="base_link" name="gripper" calibration_tool="${calibration_tool}">
     <origin xyz="0 0 0" rpy="${0 * deg_to_rad} ${-180 * deg_to_rad} 0" />
   </xacro:pal_gripper>

File: pal_gripper_description/urdf/gripper.urdf.xacro (robot description, xacro)
@@ -5,5 +5,5 @@
   <xacro:include filename="$(find pal_gripper_description)/urdf/gripper.gazebo.xacro" />
   <xacro:property name="gripper_eps" value="0.001" />
-  <xacro:macro name="pal_gripper" params="name parent *origin">
+  <xacro:macro name="pal_gripper" params="name parent *origin calibration_tool:=False">
   <link name="${name}_tool_link"/>
   <joint name="${name}_tool_joint" type="fixed">
@@ -129,10 +129,51 @@
   </joint>
   <!-- Grasping frame -->
-  <joint name="${name}_grasping_frame_joint" type="fixed">
-    <parent link="${name}_link" />
-    <child link="${name}_grasping_frame" />
-    <origin xyz="0 0 -0.13" rpy="-1.5708 1.5708 0" />
-  </joint>
-  <link name="${name}_grasping_frame"/>
+  <xacro:if value="${calibration_tool}">
+    <joint name="${name}_grasping_frame_joint" type="fixed">
+      <parent link="${name}_link" />
+      <child link="${name}_grasping_frame" />
+      <origin xyz="0 0 -0.13" rpy="-1.5708 1.5708 0" />
+    </joint>
+    <link name="${name}_grasping_frame">
+      <inertial>
+        <mass value="0.1" />
+        <origin xyz="0.21 0 0.0" rpy="0 0 0" />
+        <inertia ixx="0.000341" ixy="0" ixz="0" iyy="0.000241" iyz="0" izz="0.000101" />
+      </inertial>
+      <visual>
+        <origin xyz="0.21 0 0.0" rpy="0 0 1.5708" />
+        <geometry>
+          <box size="0.01 0.21 0.21" />
+        </geometry>
+        <material name="grasp_box_color">
+          <color rgba="0 0 1 1" />
+        </material>
+      </visual>
+      <collision>
+        <origin xyz="0.21 0 0.0" rpy="0 0 1.5708" />
+        <geometry>
+          <box size="0.01 0.21 0.21" />
+        </geometry>
+      </collision>
+    </link>
+    <gazebo reference="${name}_grasping_frame">
+      <material>Gazebo/Blue</material>
+      <turnGravityOff>true</turnGravityOff>
+    </gazebo>
+    </xacro:if>
+    <xacro:unless value="${calibration_tool}">
+      <joint name="${name}_grasping_frame_joint" type="fixed">
+        <parent link="${name}_link"/>
+        <child link="${name}_grasping_frame"/>
+        <origin xyz="0 0 -0.13" rpy="-1.5708 1.5708 0" />
+      </joint>
+      <link name="${name}_grasping_frame">
+        <inertial>
+        <mass value="0.1" />
+        <origin xyz="0.21 0 0.0" rpy="0 0 0" />
+        <inertia ixx="0.000341" ixy="0" ixz="0" iyy="0.000241" iyz="0" izz="0.000101" />
+        </inertial>
+      </link>
+    </xacro:unless>
   <xacro:finger_gazebo name="${name}_left_finger"/>
   <xacro:finger_gazebo name="${name}_right_finger"/>

Commit message: gazebo version arg missing

File: pal_gripper_description/robots/gripper_test.urdf.xacro (robot description, xacro)
@@ -31,5 +31,5 @@
   <!--Spawn gripper-->
   <link name="base_link"/>
-  <xacro:pal_gripper parent="base_link" name="gripper">
+  <xacro:pal_gripper parent="base_link" name="gripper" gazebo_version="$(arg gazebo_version)">
     <origin xyz="0 0 0" rpy="${0 * deg_to_rad} ${-180 * deg_to_rad} 0" />
   </xacro:pal_gripper>

File: pal_gripper_description/urdf/gripper.urdf.xacro (robot description, xacro)
@@ -5,5 +5,5 @@
   <xacro:include filename="$(find pal_gripper_description)/urdf/gripper.gazebo.xacro" />
   <xacro:property name="gripper_eps" value="0.001" />
-  <xacro:macro name="pal_gripper" params="name parent *origin">
+  <xacro:macro name="pal_gripper" params="name parent gazebo_version *origin">
   <link name="${name}_tool_link"/>
   <joint name="${name}_tool_joint" type="fixed">

Commit message: addition of property for gazebo_version

File: pal_gripper_description/robots/gripper_test.urdf.xacro (robot description, xacro)
@@ -18,4 +18,5 @@
   <xacro:include filename="$(find pal_gripper_description)/urdf/gripper.urdf.xacro" />
   <xacro:include filename="$(find pal_urdf_utils)/urdf/materials.urdf.xacro" />
+  <xacro:property name="gazebo_version" default="$(arg gazebo_version)"/>
   <!-- Generic simulator_gazebo plugins -->
   <!-- ros2_control -->
@@ -31,5 +32,5 @@
   <!--Spawn gripper-->
   <link name="base_link"/>
-  <xacro:pal_gripper parent="base_link" name="gripper" gazebo_version="$(arg gazebo_version)">
+  <xacro:pal_gripper parent="base_link" name="gripper">
     <origin xyz="0 0 0" rpy="${0 * deg_to_rad} ${-180 * deg_to_rad} 0" />
   </xacro:pal_gripper>

File: pal_gripper_description/urdf/gripper.urdf.xacro (robot description, xacro)
@@ -5,5 +5,5 @@
   <xacro:include filename="$(find pal_gripper_description)/urdf/gripper.gazebo.xacro" />
   <xacro:property name="gripper_eps" value="0.001" />
-  <xacro:macro name="pal_gripper" params="name parent gazebo_version *origin">
+  <xacro:macro name="pal_gripper" params="name parent *origin">
   <link name="${name}_tool_link"/>
   <joint name="${name}_tool_joint" type="fixed">
